File: darwin-integrated-panel.brd (EAGLE design)
At the start: 130 x 155 mm, 104 parts

Commit message: Cleanup.
Changed lines of the file:
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@@
 <text x="111" y="141" size="2" layer="102">PA1</text>
 <text x="12" y="12" size="2" layer="102">PA1</text>
+<hole x="5" y="140" drill="2.54"/>
+<hole x="125" y="140" drill="2.54"/>
+<hole x="5" y="15" drill="2.54"/>
+<hole x="125" y="15" drill="2.54"/>
 </plain>
 <attributes>
