File: darwin-integrated.sch (EAGLE design)
At the start: 44 parts

Commit message: Panelized. PA1.
Parts:
- added FID1, FID2, FID3, FID4, FID5, FID6: FIDUCIAL_1MM, microbuilder:FIDUCIAL_1MM
Connections:
- net MOD_G1 renamed EEPROM_PROT
- net MOD_G3 renamed HOTSWAP_INT
- removed net N$1: D1.C, RTC.VBAT, U$7.+
- removed net UPPER_PIN10: UPPER.PIN10
- new net VBACKUP: D1.C, RTC.VBAT, U$7.+, UPPER.PIN10
Changed lines of the file:
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@@
 <part name="C7" library="rcl" library_urn="urn:adsk.eagle:library:334" deviceset="C-US" device="C0603K" package3d_urn="urn:adsk.eagle:package:23680/2" value="4.7u"/>
 <part name="R5" library="rcl" library_urn="urn:adsk.eagle:library:334" deviceset="R-US_" device="R0603" package3d_urn="urn:adsk.eagle:package:23555/3"/>
+<part name="FID1" library="microbuilder" deviceset="FIDUCIAL" device="_1MM"/>
+<part name="FID2" library="microbuilder" deviceset="FIDUCIAL" device="_1MM"/>
+<part name="FID3" library="microbuilder" deviceset="FIDUCIAL" device="_1MM"/>
+<part name="FID4" library="microbuilder" deviceset="FIDUCIAL" device="_1MM"/>
+<part name="FID5" library="microbuilder" deviceset="FIDUCIAL" device="_1MM"/>
+<part name="FID6" library="microbuilder" deviceset="FIDUCIAL" device="_1MM"/>
 </parts>
 <sheets>
@@
 <attribute name="VALUE" x="120.65" y="-117.602" size="1.778" layer="96"/>
 </instance>
+<instance part="FID1" gate="G$1" x="307.34" y="-101.6" smashed="yes"/>
+<instance part="FID2" gate="G$1" x="307.34" y="-106.68" smashed="yes"/>
+<instance part="FID3" gate="G$1" x="307.34" y="-111.76" smashed="yes"/>
+<instance part="FID4" gate="G$1" x="307.34" y="-116.84" smashed="yes"/>
+<instance part="FID5" gate="G$1" x="307.34" y="-121.92" smashed="yes"/>
+<instance part="FID6" gate="G$1" x="307.34" y="-127" smashed="yes"/>
 </instances>
 <busses>
@@
 </segment>
 </net>
-<net name="MOD_G1" class="0">
+<net name="EEPROM_PROT" class="0">
 <segment>
 <pinref part="BRAIN" gate="G$2" pin="PB01"/>
@@
 </segment>
 </net>
-<net name="MOD_G3" class="0">
+<net name="HOTSWAP_INT" class="0">
 <segment>
 <pinref part="BRAIN" gate="G$2" pin="PB03"/>
@@
 </segment>
 </net>
-<net name="N$1" class="0">
+<net name="VBACKUP" class="0">
 <segment>
 <pinref part="U$7" gate="1" pin="+"/>
@@
 <wire x1="27.94" y1="-43.18" x2="7.62" y2="-43.18" width="0.1524" layer="91"/>
 <junction x="7.62" y="-43.18"/>
+<label x="12.7" y="-43.18" size="1.778" layer="95"/>
+</segment>
+<segment>
+<pinref part="UPPER" gate="G$1" pin="PIN10"/>
+<wire x1="231.14" y1="58.42" x2="210.82" y2="58.42" width="0.1524" layer="91"/>
+<label x="213.36" y="58.42" size="1.778" layer="95"/>
 </segment>
 </net>
@@
 </segment>
 </net>
-<net name="UPPER_PIN10" class="0">
-<segment>
-<pinref part="UPPER" gate="G$1" pin="PIN10"/>
-<wire x1="231.14" y1="58.42" x2="210.82" y2="58.42" width="0.1524" layer="91"/>
-<label x="213.36" y="58.42" size="1.778" layer="95"/>
-</segment>
-</net>

Commit message: Cleanup.
Parts:
- C1, C10, C11, C12, C13, C14, C15, C16, C17, C18, C19, C2, C20, C3, C4, C5, C8, C9: value (none) -> .1uf
- C23: value DSK-3R3H204T614-H2L -> .2f
- C6: value .1u -> .1uf
- C7: value 4.7u -> 4.7uf
- D1: value (none) -> VS-10BQ015HM3/5BT
- R1: value (none) -> 2k
- R2: value (none) -> 10k
- R3, R4: value (none) -> 4.7k
- R5: value (none) -> 10K
- renumbered C21 to C9, C22 to C8, U$10 to SCREEN, U$3 to U1, U$4 to U2, U$5 to U3, U$6 to U4, U$7 to C23, U$8 to USB, U$9 to SD
Other:
- note added: ".2f"
