File: darwin-upper-panel.brd (EAGLE design)
At the start: 116 x 116 mm, 104 parts, among them U1 TC58CVG1S3HRAIG, U2 TC58CVG1S3HRAIG, U3 TC58CVG1S3HRAIG, U4 TC58CVG1S3HRAIG, U5 TC58CVG1S3HRAIG, U6 TC58CVG1S3HRAIG, U7 TC58CVG1S3HRAIG, U8 TC58CVG1S3HRAIG

Commit message: Added Tag-Connect header.
Parts:
- added J1, J2: TAG-CONNECT, Conservify:TC2030-IDC
- added R11: 10K, rcl:R0603
- added R12: 10k, rcl:R0603
- R10: value 10K -> 4.7k
- R6: value 2k -> 10k
- R7: value 10k -> 2k
- R8: value 4.7k -> 10k
- moved R6 47.1 mm to (69.8, 38.9)
- moved R8 36.4 mm to (50.1, 98.9), turned to 0 degrees
- moved R10 32.8 mm to (86.5, 97.0)
- moved R7 22.9 mm to (42.5, 77.3)
- moved R9 1.50 mm to (86.5, 98.5)
Connections:
- new net SWO: J1.SWO/TDO
- new net SWO1: J2.SWO/TDO
- net 3V1: now also J2.VCC, R11.2, R12.2, R7.1; no longer R6.1, R7.2
- net 3V3: now also J1.VCC, R6.2
- net CORE_SCL1: now also R10.1; no longer R9.1
- net CORE_SDA1: now also R9.1; no longer R8.1
- net GND: now also J1.GND
- net GND1: now also J2.GND
- net N$1: now also R7.2; no longer R6.2
- net QSPI_CS1: now also R11.1; no longer R10.1
- net RESET: now also J1.NRESET
- net RESET1: now also J2.NRESET, R8.1; no longer R7.1
- net SWCLK: now also J1.SWCLK/TCK, R6.1
- net SWCLK1: now also J2.SWCLK/TCK, R12.1
- net SWDIO: now also J1.SWDIO/TMS
- net SWDIO1: now also J2.SWDIO/TMS
Routing:
- net SWCLK1: track 74.3 -> 156.7 mm, vias 0 -> 3
- net SWCLK: track 74.3 -> 156.7 mm, vias 0 -> 3
- net RESET: track 59.7 -> 89.3 mm
- net RESET1: track 59.7 -> 89.3 mm
- net SWDIO1: track 81.9 -> 110.0 mm, vias 0 -> 1
- net SWDIO: track 81.9 -> 110.0 mm, vias 0 -> 1
- net 3V3: track 73.8 -> 80.2 mm, vias 28 -> 29
- net 3V1: track 73.8 -> 80.2 mm, vias 28 -> 29
- net GND: track 51.6 -> 53.1 mm
- net GND1: track 51.6 -> 53.1 mm
Other:
- board text added: "R6"
