File: fieldkit-upper.sch (EAGLE design)
At the start: 52 parts, among them J1 TAG-CONNECT, U1 TC58CVG1S3HRAIG, U2 TC58CVG1S3HRAIG, U3 TC58CVG1S3HRAIG, U4 TC58CVG1S3HRAIG

Commit message: Schematic readability overhaul, repo look & feel.
Parts:
- C1, C10, C11, C12, C13, C14, C15, C16, C17, C18, C19, C2, C20, C3, C4, C5, C8, C9: device rcl:C-USC0603K -> Conservify:DCAP
Connections:
- net MOD_G10 renamed WIFI_RESET
- net MOD_G11 renamed WIFI_IRQ
- net MOD_G12 renamed BATTERY_CHARGING
- net MOD_G13 renamed RAD_G2
- net MOD_G14 renamed RAD_G3
- net MOD_G4 renamed WAKE_BUTTON
- net MOD_G6 renamed GPS_ENABLE
- net MOD_G7 renamed WIFI_ENABLE
- net MOD_G8 renamed WIFI_WAKE
- net MOD_G9 renamed WIFI_CS
- removed net UPPER_PIN13: UPPER.PIN13
- removed net UPPER_PIN14: UPPER.PIN14
- removed net UPPER_PIN8: UPPER.PIN8
- removed net UPPER_PIN9: UPPER.PIN9
- new net BP_ENABLE: BRAING$2.PB23, UPPER.PIN8
- new net MOD_G1: BRAING$2.PB02, LOWER.PIN13
- new net RAD_G1: BRAING$2.PB00
- net GND: now also SD.PAD1, SD.PAD2, SD.PAD3, SD.PAD4, SD.PAD5, SD.PAD6, USB.PAD1, USB.PAD2, USB.PAD3, USB.PAD4, USB.PAD5, USB.PAD6
- net MOD_G0: no longer BRAING$2.PB00
- net MOD_G2: now also BRAING$2.PB05; no longer BRAING$2.PB02, LOWER.PIN13
- net MOD_G5: no longer BRAING$2.PB05
Other:
- note added: "(Manufacturers/models/capacities vary)"
- note added: "1-4 WSON8 NAND Flash Modules"
- note added: "32KHZ from RTC ["
- note added: "ATSAMD51"
- note added: "Buttons under the screen for navigating the user interface."
- note added: "CLOCK output also drives primary clock of the ATSAMD51."
- note added: "CONNECTORS"
- note added: "Core I2C"
- note added: "D1 prevents backfeed when power is not present."
- note added: "Data Memory"
- note added: "Designed by Bradley Gawthrop for FieldKit"
- note added: "Don't watch too much, you'll rot your brain."
- note added: "Ext. Case Button ["
- note added: "Ext. Radio GPIO"
- note added: "Ext. Radio GPIO ["
- note added: "External Radio I2C"
- note added: "External Radio SPI"
- note added: "Firmware Memory"
- note added: "GPS"
- note added: "Generic 1.3" i2C OLED Module."
- note added: "Inrush/Charging Current limited by R1"
- note added: "Interrupt for Module Insert/Remove ["
- note added: "JTAG"
- note added: "Module EEPROM Reserved/Ready ["
- note added: "Module GPIO ["
- note added: "Module I2C"
- note added: "Navigation Buttons"
- note added: "OLED Display"
- note added: "PCF85363"
- note added: "PERIPHERALS"
- note added: "Peripheral Power"
- note added: "RTC"
- note added: "Real-Time Clock"
- note added: "SD Card"
- note added: "Temperature Sensor"
- note added: "Temperature inside the FieldKit enclosure is logged"
- note added: "User Buttons"
- note added: "VBACKUP Provided by supercap C23"
- note added: "Wiifi Module"
- note added: "] 'Backpack' Module Enable"
- note added: "biased by internal pull-ups on the ATSAMD51."
- note added: "mostly to predict battery health in the cold."
- note removed: "BUTTONS"
- note removed: "CLOCK"
- note removed: "DECOUPLING"
- note removed: "MCU"
- note removed: "MEMORY"
- note removed: "MEZZANINE"
- note removed: "PROGRAMMING HEADER"
- note removed: "SCREEN"
- note removed: "SD CARD"
- note removed: "TEMP"
